Commit message: fixed front wheel not showing up

File: isaac_ros-dev/src/agv_car_description/description/ros2_control_ackerman.xacro (robot description, xacro)
@@ -23,4 +23,10 @@
       <state_interface name="position" />
     </joint>
+    <joint name="front_right_wheel_joint">
+      <state_interface name="position" />
+    </joint>
+    <joint name="front_left_wheel_joint">
+      <state_interface name="position" />
+    </joint>
   </ros2_control>
   <gazebo>
