Commit message: making it work with ros2 control using ackerman

File: isaac_ros-dev/src/agv_car_description/description/agv_car.xacro (robot description, xacro)
@@ -14,5 +14,5 @@
     <link name="base_link">
         <visual>
-            <origin xyz=".946 .521 -.313" rpy="0 0 ${pi}" />
+            <origin xyz=".946 .521 -0.313" rpy="0 0 ${pi}" />
             <geometry>
                 <mesh filename="package://agv_car_gazebo/models/agv_car/meshes/agv_chassis.stl"/>
@@ -49,5 +49,5 @@
             </visual>
             <collision>
-                <origin xyz="0 0 0" rpy="${pi/2} 0 0"/>
+                <!-- <origin xyz="0 0 0" rpy="${pi/2} 0 0"/> -->
                 <geometry>
                     <cylinder radius="${wheel_radius}" length="${wheel_width}"/>
@@ -59,5 +59,5 @@
             <parent link="base_link"/>
             <child link="rear_${prefix}_wheel"/>
-            <origin xyz="${x_reflect*wheel_xoff} ${y_reflect*(base_width/2+wheel_ygap)} ${-wheel_zoff}" rpy="0 0 0"/>
+            <origin xyz="${x_reflect*wheel_xoff} ${y_reflect*(base_width/2+wheel_ygap)} 0" rpy="0 0 0"/>
             <axis xyz="0 0 1"/>
             <limit effort="1000.0" lower="-0.698" upper="0.698" velocity="0.5"/>
@@ -88,5 +88,5 @@
             <parent link="base_link"/>
             <child link="front_${prefix}_steering_wheel_link"/>
-            <origin xyz="${x_reflect * wheel_xoff} ${y_reflect * (base_width / 2 + wheel_ygap)} ${-wheel_zoff}" rpy="0 0 0"/>
+            <origin xyz="${x_reflect * wheel_xoff} ${y_reflect * (base_width / 2 + wheel_ygap)} 0" rpy="0 0 0"/>
             <axis xyz="0 0 1"/>
             <limit effort="1000.0" lower="-0.698" upper="0.698" velocity="0.5"/>
@@ -108,4 +108,5 @@
             </visual>
             <collision>
+                <!-- <origin xyz="0 0 0" rpy="${pi/2} 0 0"/> -->
                 <geometry>
                     <cylinder radius="${wheel_radius}" length="${wheel_width}"/>
@@ -137,5 +138,5 @@
     <parent link="base_link"/>
     <child link="virtual_front_wheel"/>
-    <origin xyz="${wheel_xoff} 0 ${-wheel_zoff}" rpy="0 0 ${pi/2}"/>
+    <origin xyz="${wheel_xoff} 0 0" rpy="0 0 ${pi/2}"/>
     <axis xyz="0 0 1"/>
     <limit lower="-0.7853" upper="0.7853" effort="100.0" velocity="100.0"/>
@@ -155,5 +156,5 @@
     <parent link="base_link"/>
     <child link="virtual_rear_wheel"/>
-    <origin xyz="${-wheel_xoff} 0 ${-wheel_zoff}" rpy="0 0 ${pi/2}"/>
+    <origin xyz="${-wheel_xoff} 0 0" rpy="0 0 ${pi/2}"/>
     <axis xyz="1 0 0"/>
     <limit effort="100.0" velocity="100.0"/>

File: isaac_ros-dev/src/agv_car_description/description/final_agv_car.xacro (robot description, xacro)
@@ -1,5 +1,6 @@
 <?xml version="1.0"?>
 <robot name="my_robot" xmlns:xacro="http://www.ros.org/wiki/xacro">
-  <xacro:include filename="agv_car.xacro" />
+  <!-- <xacro:include filename="agv_car.xacro" /> -->
+  <xacro:include filename="test.xacro" />
   <xacro:include filename="ros2_control_ackerman.xacro" />
   <!-- <xacro:include filename="ros2_control_bicycle.xacro" /> -->

File: isaac_ros-dev/src/agv_car_description/description/ros2_control_ackerman.xacro (robot description, xacro)
@@ -1,54 +1,30 @@
 <?xml version="1.0"?>
 <robot xmlns:xacro="http://www.ros.org/wiki/xacro">
-    <ros2_control name="GazeboSystem" type="system">
-        <hardware>
-            <plugin>gazebo_ros2_control/GazeboSystem</plugin>
-        </hardware>
-        <joint name="left_rear_wheel_joint">
-            <command_interface name="velocity">
-                <param name="min">-10.0</param>
-                <param name="max">10.0</param>
-            </command_interface>
-            <state_interface name="velocity"/>
-            <state_interface name="position"/>
-        </joint>
-        <joint name="right_rear_wheel_joint">
-            <command_interface name="velocity">
-                <param name="min">-10.0</param>
-                <param name="max">10.0</param>
-            </command_interface>
-            <state_interface name="velocity"/>
-            <state_interface name="position"/>
-        </joint>
-        <joint name="left_front_steering_joint">
-            <command_interface name="velocity">
-                <param name="min">-1.0</param>
-                <param name="max">1.0</param>
-            </command_interface>
-            <command_interface name="position"/>
-            <state_interface name="velocity"/>
-            <state_interface name="position"/>
-        </joint>
-        <joint name="right_front_steering_joint">
-            <command_interface name="velocity">
-                <param name="min">-1.0</param>
-                <param name="max">1.0</param>
-            </command_interface>
-            <command_interface name="position"/>
-            <state_interface name="velocity"/>
-            <state_interface name="position"/>
-        </joint>
-        <joint name="left_front_wheel_joint">
-            <!-- <command_interface name="position"/> -->
-            <state_interface name="position"/>
-        </joint>
-        <joint name="right_front_wheel_joint">
-            <!-- <command_interface name="position"/> -->
-            <state_interface name="position"/>
-        </joint>
-    </ros2_control>
+    <ros2_control name="IgnitionSystem" type="system">
+    <hardware>
+      <plugin>ign_ros2_control/IgnitionSystem</plugin>
+    </hardware>
+    <joint name="rear_left_wheel_joint">
+      <command_interface name="velocity" />
+      <state_interface name="velocity" />
+      <state_interface name="position" />
+    </joint>
+    <joint name="rear_right_wheel_joint">
+      <command_interface name="velocity" />
+      <state_interface name="velocity" />
+      <state_interface name="position" />
+    </joint>
+    <joint name="left_wheel_steering_joint">
+      <command_interface name="position" />
+      <state_interface name="position" />
+    </joint>
+    <joint name="right_wheel_steering_joint">
+      <command_interface name="position" />
+      <state_interface name="position" />
+    </joint>
+  </ros2_control>
     <gazebo>
-        <plugin name="gazebo_ros2_control" filename="libgazebo_ros2_control.so">
-            <parameters>$(find agv_car_description)/config/controllers.yaml</parameters>
+        <plugin filename="ign_ros2_control-system" name="ign_ros2_control::IgnitionROS2ControlPlugin">
+        <parameters>$(find agv_car_description)/config/controllers.yaml</parameters>
         </plugin>
     </gazebo>

Commit message: changes to make rviz work

File: isaac_ros-dev/src/agv_car_description/description/agv_car.xacro (robot description, xacro)
@@ -22,5 +22,7 @@
             </material>
         </visual>
+\
         <collision>
+            <origin xyz=".946 .521 -0.313" rpy="0 0 ${pi}" />
             <geometry>
                 <mesh filename="package://agv_car_gazebo/models/agv_car/meshes/agv_chassis.stl"/>

File: isaac_ros-dev/src/agv_car_description/description/test.xacro (robot description, xacro)
@@ -34,8 +34,8 @@
         </visual>
         <collision>
-            <origin xyz="0 0 0" rpy="0 0 0" />
-            <geometry>
-                <mesh filename="package://agv_car_gazebo/models/agv_car/meshes/agv_chassis.stl"/>
-            </geometry>
+            <origin xyz=".946 .521 -0.313" rpy="0 0 ${pi}" />
+                <geometry>
+                    <mesh filename="package://agv_car_gazebo/models/agv_car/meshes/agv_chassis.stl"/>
+                </geometry>
         </collision>
         <!-- <xacro:box_inertia m="15" w="${base_width}" d="${base_length}" h="${base_height}"/> -->
@@ -189,3 +189,20 @@
         <dynamics damping="0.2" />
     </joint>
+        <!-- Lidar -->
+    <link name="velodyne">
+        <visual>
+            <origin xyz="0 0 0" rpy="0 0 0"/>
+            <geometry>
+                <cylinder radius=".0762" length=".0762"/>
+            </geometry>
+            <material name="Cyan">
+                <color rgba="0 1.0 1.0 1.0"/>
+            </material>
+        </visual>
+    </link>
+    <joint name="velodyne_joint" type="fixed">
+        <parent link="base_link"/>
+        <child link="velodyne"/>
+        <origin xyz="0 0 1.0414" rpy="0 0 0"/>
+    </joint>
 </robot>
