Commit message: changes to  run bicycle controller initially

File: isaac_ros-dev/src/agv_car_description/description/agv_car.xacro (robot description, xacro)
@@ -1,6 +1,4 @@
 <?xml version="1.0"?>
-<robot name="new_car" xmlns:xacro="http://ros.org/wiki/xacro">
-    <!-- <xacro:include filename="colors.xacro" /> -->
-    <xacro:include filename="inertial_macros.xacro" />
+<robot name="ackermann_drive" xmlns:xacro="http://ros.org/wiki/xacro">
     <xacro:property name="base_width" value="1.041"/>
     <xacro:property name="base_length" value="1.892"/>
@@ -11,9 +9,22 @@
     <xacro:property name="wheel_zoff" value="0.123"/>
     <xacro:property name="wheel_xoff" value="0.756"/>
-    <!-- Robot Base -->
-    <link name="base_link">
-        <visual>
-            <origin xyz=".946 .521 -0.313" rpy="0 0 ${pi}" />
-            <geometry>
+    <material name="Black">
+    <color rgba="0 0 0 1" />
+    </material>
+    <material name="Grey">
+        <color rgba="0.8 0.8 0.8 1" />
+    </material>
+    <material name="Orange">
+        <color rgba="1 0.6 0 1" />
+    </material>
+    <material name="White">
+        <color rgba="1 1 1 1" />
+    </material>
+    <link name="base_link" />
+    <!-- Chassis -->
+    <link name="chassis">
+        <visual>
+        <origin xyz=".946 .521 -0.313" rpy="0 0 ${pi}" />
+         <geometry>
                 <mesh filename="package://agv_car_gazebo/models/agv_car/meshes/agv_chassis.stl"/>
             </geometry>
@@ -24,108 +35,159 @@
         <collision>
             <origin xyz=".946 .521 -0.313" rpy="0 0 ${pi}" />
-            <geometry>
-                <mesh filename="package://agv_car_gazebo/models/agv_car/meshes/agv_chassis.stl"/>
-            </geometry>
+                <geometry>
+                    <mesh filename="package://agv_car_gazebo/models/agv_car/meshes/agv_chassis.stl"/>
+                </geometry>
         </collision>
-        <xacro:box_inertia m="15" w="${base_width}" d="${base_length}" h="${base_height}"/>
-    </link>
-    <!-- Robot Footprint -->
-    <link name="base_footprint"/>
-    <joint name="base_joint" type="fixed">
-        <parent link="base_link"/>
-        <child link="base_footprint"/>
-        <origin xyz="0.0 0.0 ${-(wheel_radius+wheel_zoff)}" rpy="0 0 0"/>
-    </joint>
-    <!-- Wheels -->
-    <xacro:macro name="rearwheel" params="prefix x_reflect y_reflect">
-        <link name="rear_${prefix}_wheel">
-            <visual>
-                <origin xyz="0 0 0" rpy="${pi/2} 0 0"/>
-                <geometry>
-                    <cylinder radius="${wheel_radius}" length="${wheel_width}"/>
-                </geometry>
-                <material name="Gray">
-                    <color rgba="0.5 0.5 0.5 1.0"/>
-                </material>
-            </visual>
-            <collision>
-                <!-- <origin xyz="0 0 0" rpy="${pi/2} 0 0"/> -->
-                <geometry>
-                    <cylinder radius="${wheel_radius}" length="${wheel_width}"/>
-                </geometry>
-            </collision>
-            <xacro:cylinder_inertia m="0.5" r="${wheel_radius}" h="${wheel_width}"/>
-        </link>
-        <joint name="rear_${prefix}_wheel_joint" type="revolute">
-            <parent link="base_link"/>
-            <child link="rear_${prefix}_wheel"/>
-            <origin xyz="${x_reflect*wheel_xoff} ${y_reflect*(base_width/2+wheel_ygap)} 0" rpy="0 0 0"/>
-            <axis xyz="0 0 1"/>
-            <limit effort="1000.0" lower="-0.698" upper="0.698" velocity="0.5"/>
-        </joint>
-    </xacro:macro>
-    <xacro:rearwheel prefix="left" x_reflect="-1" y_reflect="1"/>
-    <xacro:rearwheel prefix="right" x_reflect="-1" y_reflect="-1"/>
-    <!-- Steering Wheels -->
-    <xacro:macro name="steering_wheel" params="prefix x_reflect y_reflect">
-        <link name="front_${prefix}_steering_wheel_link">
-            <visual>
-                <origin xyz="0.05 ${y_reflect * (wheel_width / 2 - .1)} 0" rpy="${pi/2} ${pi/2} 0"/>
-                <geometry>
-                    <cylinder radius="0.029999999" length="0.1000000"/>
-                </geometry>
-                <material name="Gray">
-                    <color rgba="0.5 0.5 0.5 1.0"/>
-                </material>
-            </visual>
-            <collision>
-                <geometry>
-                    <cylinder radius="0.029999999" length="0.10000000"/>
-                </geometry>
-            </collision>
-            <xacro:cylinder_inertia m="0.5" r="${wheel_radius}" h="${wheel_width}"/>
-        </link>
-        <joint name="front_${prefix}_wheel_steering_joint" type="revolute">
-            <parent link="base_link"/>
-            <child link="front_${prefix}_steering_wheel_link"/>
-            <origin xyz="${x_reflect * wheel_xoff} ${y_reflect * (base_width / 2 + wheel_ygap)} 0" rpy="0 0 0"/>
-            <axis xyz="0 0 1"/>
-            <limit effort="1000.0" lower="-0.698" upper="0.698" velocity="0.5"/>
-        </joint>
-    </xacro:macro>
-    <xacro:steering_wheel prefix="left" x_reflect="1" y_reflect="1"/>
-    <xacro:steering_wheel prefix="right" x_reflect="1" y_reflect="-1"/>
-    <!-- Front Wheels -->
-    <xacro:macro name="frontwheel" params="prefix x_reflect y_reflect">
-        <link name="front_${prefix}_wheel">
-            <visual>
-                <origin xyz="0 0 0" rpy="${pi/2} 0 0"/>
-                <geometry>
-                    <cylinder radius="${wheel_radius}" length="${wheel_width}"/>
-                </geometry>
-                <material name="Gray">
-                    <color rgba="0.5 0.5 0.5 1.0"/>
-                </material>
-            </visual>
-            <collision>
-                <!-- <origin xyz="0 0 0" rpy="${pi/2} 0 0"/> -->
-                <geometry>
-                    <cylinder radius="${wheel_radius}" length="${wheel_width}"/>
-                </geometry>
-            </collision>
-            <xacro:cylinder_inertia m="0.5" r="${wheel_radius}" h="${wheel_width}"/>
-        </link>
-        <joint name="front_${prefix}_wheel_joint" type="revolute">
-            <parent link="front_${prefix}_steering_wheel_link"/>
-            <child link="front_${prefix}_wheel"/>
-            <origin xyz="0 0 0" rpy="0 0 0"/>
-            <axis xyz="0 0 1"/>
-            <limit effort="1000.0" lower="-0.698" upper="0.698" velocity="0.5"/>
-        </joint>
-    </xacro:macro>
-    <xacro:frontwheel prefix="left" x_reflect="1" y_reflect="1"/>
-    <xacro:frontwheel prefix="right" x_reflect="1" y_reflect="-1"/>
-        <!-- virtual front wheel -->
-    <link name="virtual_front_wheel">
+        <!-- <xacro:box_inertia m="15" w="${base_width}" d="${base_length}" h="${base_height}"/> -->
+        <inertial>
+        <origin xyz="0 0 0" rpy="0 0 0" />
+        <mass value="100" />
+        <inertia ixx="10.4" ixy="0.0" ixz="0.0" iyy="35.4" iyz="0.0" izz="41.66" />
+        </inertial>
+    </link>
+    <joint name="chassis_joint" type="fixed">
+        <origin xyz="0.8 0 0.5" rpy="0 0 0" />
+        <parent link="base_link" />
+        <child link="chassis" />
+    </joint>
+    <!-- rear left wheel Link -->
+    <link name="rear_left_wheel">
+        <visual>
+            <geometry>
+                <cylinder radius="${wheel_radius}" length="${wheel_width}"/>
+            </geometry>
+            <material name="Gray">
+                <color rgba="0.5 0.5 0.5 1.0"/>
+            </material>
+        </visual>
+            <collision>
+                <geometry>
+                    <cylinder radius="${wheel_radius}" length="${wheel_width}"/>
+                </geometry>
+            </collision>
+        <inertial>
+        <mass value="11.3" />
+        <inertia ixx="0.26" ixy="0.0" ixz="0.0" iyy="0.26" iyz="0.0" izz="0.51" />
+        </inertial>
+    </link>
+    <joint name="rear_left_wheel_joint" type="continuous">
+        <origin xyz="-0.8 0.5 -0.2" rpy="-1.57 0 0" />
+        <parent link="chassis" />
+        <child link="rear_left_wheel" />
+        <axis xyz="0 0 1" />
+        <dynamics damping="0.2" />
+    </joint>
+    <!-- rear right wheel Link -->
+    <link name="rear_right_wheel">
+        <visual>
+            <geometry>
+                <cylinder radius="${wheel_radius}" length="${wheel_width}"/>
+            </geometry>
+            <material name="Gray">
+                <color rgba="0.5 0.5 0.5 1.0"/>
+            </material>
+        </visual>
+            <collision>
+                <geometry>
+                    <cylinder radius="${wheel_radius}" length="${wheel_width}"/>
+                </geometry>
+            </collision>
+        <inertial>
+        <mass value="11.3" />
+        <inertia ixx="0.26" ixy="0.0" ixz="0.0" iyy="0.26" iyz="0.0" izz="0.51" />
+        </inertial>
+    </link>
+    <joint name="rear_right_wheel_joint" type="continuous">
+        <origin xyz="-0.8 -0.5 -0.2" rpy="-1.57 0 0" />
+        <parent link="chassis" />
+        <child link="rear_right_wheel" />
+        <axis xyz="0 0 1" />
+        <dynamics damping="0.2" />
+    </joint>
+    <!-- left steer Link -->
+    <link name="left_wheel_steering">
+        <inertial>
+        <mass value="0.1"/>
+        <inertia ixx="0" ixy="0.0" ixz="0.0" iyy="0.0" iyz="0.0" izz="0.0" />
+        </inertial>
+    </link>
+    <joint name="left_wheel_steering_joint" type="revolute">
+        <origin xyz="0.9 0.5 -0.2" rpy="1.57 0 0" />
+        <parent link="chassis" />
+        <child link="left_wheel_steering" />
+        <axis xyz="0 1 0" />
+        <dynamics damping="0.2" />
+        <limit effort="1000.0" lower="-1.57" upper="1.57" velocity="30"/>
+    </joint>
+    <!-- right steer Link -->
+    <link name="right_wheel_steering">
+        <inertial>
+        <mass value="0.1"/>
+        <inertia ixx="0" ixy="0.0" ixz="0.0" iyy="0.0" iyz="0.0" izz="0.0" />
+        </inertial>
+    </link>
+    <joint name="right_wheel_steering_joint" type="revolute">
+        <origin xyz="0.9 -0.5 -0.2" rpy="1.57 0 0" />
+        <parent link="chassis" />
+        <child link="right_wheel_steering" />
+        <axis xyz="0 1 0" />
+        <dynamics damping="0.2" />
+        <limit effort="1000.0" lower="-1.57" upper="1.57" velocity="30"/>
+    </joint>
+    <!-- front left wheel Link -->
+    <link name="front_left_wheel">
+         <visual>
+            <geometry>
+                <cylinder radius="${wheel_radius}" length="${wheel_width}"/>
+            </geometry>
+            <material name="Gray">
+                <color rgba="0.5 0.5 0.5 1.0"/>
+            </material>
+        </visual>
+            <collision>
+                <geometry>
+                    <cylinder radius="${wheel_radius}" length="${wheel_width}"/>
+                </geometry>
+            </collision>
+        <inertial>
+        <mass value="11.3" />
+        <inertia ixx="0.26" ixy="0.0" ixz="0.0" iyy="0.26" iyz="0.0" izz="0.51" />
+        </inertial>
+    </link>
+    <joint name="front_left_wheel_joint" type="continuous">
+        <origin xyz="0 0 0" rpy="0 0 0" />
+        <parent link="left_wheel_steering" />
+        <child link="front_left_wheel" />
+        <axis xyz="0 0 1" />
+        <dynamics damping="0.2" />
+    </joint>
+    <!-- front right wheel Link -->
+    <link name="front_right_wheel">
+        <visual>
+            <geometry>
+                <cylinder radius="${wheel_radius}" length="${wheel_width}"/>
+            </geometry>
+            <material name="Gray">
+                <color rgba="0.5 0.5 0.5 1.0"/>
+            </material>
+        </visual>
+            <collision>
+                <geometry>
+                    <cylinder radius="${wheel_radius}" length="${wheel_width}"/>
+                </geometry>
+            </collision>
+        <inertial>
+        <mass value="11.3" />
+        <inertia ixx="0.26" ixy="0.0" ixz="0.0" iyy="0.26" iyz="0.0" izz="0.51" />
+        </inertial>
+    </link>
+    <joint name="front_right_wheel_joint" type="continuous">
+        <origin xyz="0 0 0" rpy="0 0 0" />
+        <parent link="right_wheel_steering" />
+        <child link="front_right_wheel" />
+        <axis xyz="0 0 1" />
+        <dynamics damping="0.2" />
+    </joint>
+     <link name="virtual_front_wheel">
     <visual>
         <origin xyz="0 0 0" rpy="${pi/2} 0 ${pi/2}"/>
@@ -133,5 +195,5 @@
         <cylinder length="0.01" radius="${wheel_radius}"/>
         </geometry>
-        <material name="invisible"/>
+        <!-- <material name="invisible"/> -->
     </visual>
     </link>
@@ -151,5 +213,5 @@
         <cylinder length="0.01" radius="${wheel_radius}"/>
         </geometry>
-        <material name="invisible"/>
+        <!-- <material name="invisible"/> -->
     </visual>
     </link>
@@ -162,5 +224,5 @@
     <dynamics damping="0.2"/>
     </joint>
-    <!-- Lidar -->
+        <!-- Lidar -->
     <link name="velodyne">
         <visual>
@@ -175,5 +237,5 @@
     </link>
     <joint name="velodyne_joint" type="fixed">
-        <parent link="base_link"/>
+        <parent link="chassis"/>
         <child link="velodyne"/>
         <origin xyz="0 0 1.0414" rpy="0 0 0"/>

File: isaac_ros-dev/src/agv_car_description/description/final_agv_car.xacro (robot description, xacro)
@@ -1,8 +1,8 @@
 <?xml version="1.0"?>
 <robot name="my_robot" xmlns:xacro="http://www.ros.org/wiki/xacro">
-  <!-- <xacro:include filename="agv_car.xacro" /> -->
-  <xacro:include filename="test.xacro" />
-  <xacro:include filename="ros2_control_ackerman.xacro" />
-  <!-- <xacro:include filename="ros2_control_bicycle.xacro" /> -->
+  <xacro:include filename="agv_car.xacro" />
+  <!-- <xacro:include filename="test.xacro" /> -->
+  <!-- <xacro:include filename="ros2_control_ackerman.xacro" /> -->
+  <xacro:include filename="ros2_control_bicycle.xacro" />
   <!-- <xacro:include filename="lidar.xacro" />
   <xacro:include filename="depth_camera.xacro" /> -->

File: isaac_ros-dev/src/agv_car_description/description/ros2_control_bicycle.xacro (robot description, xacro)
@@ -3,10 +3,10 @@
     <ros2_control name="RobotControl" type="system">
         <hardware>
-            <plugin>bicdrive_arduino/CarlikeBotSystemHardware</plugin>
+            <plugin>arduino_car_hardware/CarlikeBotSystemHardware</plugin>
             <param name="front_wheel_name">virtual_front_wheel_joint</param>
             <param name="rear_wheel_name">virtual_rear_wheel_joint</param>
             <param name="loop_rate">30</param>
-            <param name="device">/dev/serial/by-id/usb-1a86_USB2.0-Ser_-if00-port0</param>
-            <param name="baud_rate">9600</param>
+            <param name="device">/dev/ttyACM0</param>
+            <param name="baud_rate">115200</param>
             <param name="timeout_ms">1000</param>
         </hardware>
@@ -18,5 +18,4 @@
             <command_interface name="velocity"/>
             <state_interface name="velocity"/>
-            <state_interface name="position"/>
         </joint>
     </ros2_control>

File: isaac_ros-dev/src/agv_car_description/description/test.xacro (robot description, xacro)
@@ -189,4 +189,39 @@
         <dynamics damping="0.2" />
     </joint>
+     <link name="virtual_front_wheel">
+    <visual>
+        <origin xyz="0 0 0" rpy="${pi/2} 0 ${pi/2}"/>
+        <geometry>
+        <cylinder length="0.01" radius="${wheel_radius}"/>
+        </geometry>
+        <material name="invisible"/>
+    </visual>
+    </link>
+    <joint name="virtual_front_wheel_joint" type="revolute">
+    <parent link="base_link"/>
+    <child link="virtual_front_wheel"/>
+    <origin xyz="${wheel_xoff} 0 0" rpy="0 0 ${pi/2}"/>
+    <axis xyz="0 0 1"/>
+    <limit lower="-0.7853" upper="0.7853" effort="100.0" velocity="100.0"/>
+    <dynamics damping="0.2"/>
+    </joint>
+    <!-- virtual rear wheel -->
+    <link name="virtual_rear_wheel">
+    <visual>
+        <origin xyz="0 0 0" rpy="${pi/2} 0 ${pi/2}"/>
+        <geometry>
+        <cylinder length="0.01" radius="${wheel_radius}"/>
+        </geometry>
+        <material name="invisible"/>
+    </visual>
+    </link>
+    <joint name="virtual_rear_wheel_joint" type="continuous">
+    <parent link="base_link"/>
+    <child link="virtual_rear_wheel"/>
+    <origin xyz="${-wheel_xoff} 0 0" rpy="0 0 ${pi/2}"/>
+    <axis xyz="1 0 0"/>
+    <limit effort="100.0" velocity="100.0"/>
+    <dynamics damping="0.2"/>
+    </joint>
         <!-- Lidar -->
     <link name="velodyne">

Commit message: changes to fix car odometry and urdf

File: isaac_ros-dev/src/agv_car_description/description/agv_car.xacro (robot description, xacro)
@@ -25,7 +25,7 @@
     <link name="chassis">
         <visual>
-        <origin xyz=".946 .521 -0.313" rpy="0 0 ${pi}" />
+        <origin xyz="0 0 -0.313" rpy="0 0 ${pi}" />
          <geometry>
-                <mesh filename="package://agv_car_gazebo/models/agv_car/meshes/agv_chassis.stl"/>
+                <mesh filename="package://agv_car_description/meshes/agv_chassis.stl"/>
             </geometry>
             <material name="Cyan">
@@ -36,5 +36,5 @@
             <origin xyz=".946 .521 -0.313" rpy="0 0 ${pi}" />
                 <geometry>
-                    <mesh filename="package://agv_car_gazebo/models/agv_car/meshes/agv_chassis.stl"/>
+                    <mesh filename="package://agv_car_description/meshes/agv_chassis.stl"/>
                 </geometry>
         </collision>
@@ -47,5 +47,5 @@
     </link>
     <joint name="chassis_joint" type="fixed">
-        <origin xyz="0.8 0 0.5" rpy="0 0 0" />
+        <origin xyz="0 0 0.5" rpy="0 0 0" />
         <parent link="base_link" />
         <child link="chassis" />

Commit message: changes to fix urdf

File: isaac_ros-dev/src/agv_car_description/description/agv_car.xacro (robot description, xacro)
@@ -25,5 +25,5 @@
     <link name="chassis">
         <visual>
-        <origin xyz="0 0 -0.313" rpy="0 0 ${pi}" />
+        <origin xyz=".946 .512 -.313" rpy="0 0 ${pi}" />
          <geometry>
                 <mesh filename="package://agv_car_description/meshes/agv_chassis.stl"/>
@@ -34,5 +34,5 @@
         </visual>
         <collision>
-            <origin xyz=".946 .521 -0.313" rpy="0 0 ${pi}" />
+            <origin xyz=".946 .512 -.313" rpy="0 0 ${pi}" />
                 <geometry>
                     <mesh filename="package://agv_car_description/meshes/agv_chassis.stl"/>
@@ -47,5 +47,5 @@
     </link>
     <joint name="chassis_joint" type="fixed">
-        <origin xyz="0 0 0.5" rpy="0 0 0" />
+        <origin xyz="0 0 .313" rpy="0 0 0" />
         <parent link="base_link" />
         <child link="chassis" />
@@ -72,5 +72,5 @@
     </link>
     <joint name="rear_left_wheel_joint" type="continuous">
-        <origin xyz="-0.8 0.5 -0.2" rpy="-1.57 0 0" />
+        <origin xyz="-0.9 0.5 -0.2" rpy="-1.57 0 0" />
         <parent link="chassis" />
         <child link="rear_left_wheel" />
@@ -99,5 +99,5 @@
     </link>
     <joint name="rear_right_wheel_joint" type="continuous">
-        <origin xyz="-0.8 -0.5 -0.2" rpy="-1.57 0 0" />
+        <origin xyz="-0.9 -0.5 -0.2" rpy="-1.57 0 0" />
         <parent link="chassis" />
         <child link="rear_right_wheel" />
@@ -191,5 +191,5 @@
      <link name="virtual_front_wheel">
     <visual>
-        <origin xyz="0 0 0" rpy="${pi/2} 0 ${pi/2}"/>
+        <origin xyz="0 0 0" py="0 0 0"/>
         <geometry>
         <cylinder length="0.01" radius="${wheel_radius}"/>
@@ -199,7 +199,7 @@
     </link>
     <joint name="virtual_front_wheel_joint" type="revolute">
-    <parent link="base_link"/>
+    <parent link="chassis"/>
     <child link="virtual_front_wheel"/>
-    <origin xyz="${wheel_xoff} 0 0" rpy="0 0 ${pi/2}"/>
+    <origin xyz="0.9 0 -0.2" rpy="1.57 0 0"/>
     <axis xyz="0 0 1"/>
     <limit lower="-0.7853" upper="0.7853" effort="100.0" velocity="100.0"/>
@@ -209,5 +209,5 @@
     <link name="virtual_rear_wheel">
     <visual>
-        <origin xyz="0 0 0" rpy="${pi/2} 0 ${pi/2}"/>
+        <origin xyz="0 0 0" rpy="0 0 0"/>
         <geometry>
         <cylinder length="0.01" radius="${wheel_radius}"/>
@@ -217,8 +217,8 @@
     </link>
     <joint name="virtual_rear_wheel_joint" type="continuous">
-    <parent link="base_link"/>
+    <parent link="chassis"/>
     <child link="virtual_rear_wheel"/>
-    <origin xyz="${-wheel_xoff} 0 0" rpy="0 0 ${pi/2}"/>
-    <axis xyz="1 0 0"/>
+    <origin xyz="-0.9 0 -0.2" rpy="-1.57 0 0"/>
+    <axis xyz="0 0 1"/>
     <limit effort="100.0" velocity="100.0"/>
     <dynamics damping="0.2"/>

Commit message: changes to fix odometry and visual in rviz, next step is nav2 setup

File: isaac_ros-dev/src/agv_car_description/description/agv_car.xacro (robot description, xacro)
@@ -191,5 +191,5 @@
      <link name="virtual_front_wheel">
     <visual>
-        <origin xyz="0 0 0" py="0 0 0"/>
+        <origin xyz="0 0 0" rpy="0 0 0"/>
         <geometry>
         <cylinder length="0.01" radius="${wheel_radius}"/>
@@ -202,5 +202,5 @@
     <child link="virtual_front_wheel"/>
     <origin xyz="0.9 0 -0.2" rpy="1.57 0 0"/>
-    <axis xyz="0 0 1"/>
+    <axis xyz="0 1 0"/>
     <limit lower="-0.7853" upper="0.7853" effort="100.0" velocity="100.0"/>
     <dynamics damping="0.2"/>

Commit message: changes for fixing navsat node

File: isaac_ros-dev/src/agv_car_description/description/agv_car.xacro (robot description, xacro)
@@ -224,6 +224,21 @@
     <dynamics damping="0.2"/>
     </joint>
+        <!-- IMU and GPS combined sensor -->
+    <link name="imu_link"/>
+    <joint name="imu_joint" type="fixed">
+    <parent link="chassis"/>
+    <child link="imu_link"/>
+    <!-- Adjust this to the actual mounting point on your robot -->
+    <origin xyz="0 0 1.2" rpy="0 0 0"/>
+    </joint>
+    <link name="gps_link"/>
+    <joint name="gps_joint" type="fixed">
+    <parent link="chassis"/>
+    <child link="gps_link"/>
+    <!-- Same origin as imu_link -->
+    <origin xyz="0 0 1.2" rpy="0 0 0"/>
+    </joint>
         <!-- Lidar -->
-    <link name="velodyne">
+    <link name="lidar">
         <visual>
             <origin xyz="0 0 0" rpy="0 0 0"/>
@@ -236,7 +251,7 @@
         </visual>
     </link>
-    <joint name="velodyne_joint" type="fixed">
+    <joint name="lidar_joint" type="fixed">
         <parent link="chassis"/>
-        <child link="velodyne"/>
+        <child link="lidar"/>
         <origin xyz="0 0 1.0414" rpy="0 0 0"/>
     </joint>
