Commit message: changes to make navsat work finally but with yaw issue

File: isaac_ros-dev/src/agv_car_description/description/agv_car.xacro (robot description, xacro)
@@ -71,5 +71,5 @@
         </inertial>
     </link>
-    <joint name="rear_left_wheel_joint" type="continuous">
+    <joint name="rear_left_wheel_joint" type="fixed">
         <origin xyz="-0.9 0.5 -0.2" rpy="-1.57 0 0" />
         <parent link="chassis" />
@@ -98,5 +98,5 @@
         </inertial>
     </link>
-    <joint name="rear_right_wheel_joint" type="continuous">
+    <joint name="rear_right_wheel_joint" type="fixed">
         <origin xyz="-0.9 -0.5 -0.2" rpy="-1.57 0 0" />
         <parent link="chassis" />
@@ -112,5 +112,5 @@
         </inertial>
     </link>
-    <joint name="left_wheel_steering_joint" type="revolute">
+    <joint name="left_wheel_steering_joint" type="fixed">
         <origin xyz="0.9 0.5 -0.2" rpy="1.57 0 0" />
         <parent link="chassis" />
@@ -127,5 +127,5 @@
         </inertial>
     </link>
-    <joint name="right_wheel_steering_joint" type="revolute">
+    <joint name="right_wheel_steering_joint" type="fixed">
         <origin xyz="0.9 -0.5 -0.2" rpy="1.57 0 0" />
         <parent link="chassis" />
@@ -155,5 +155,5 @@
         </inertial>
     </link>
-    <joint name="front_left_wheel_joint" type="continuous">
+    <joint name="front_left_wheel_joint" type="fixed">
         <origin xyz="0 0 0" rpy="0 0 0" />
         <parent link="left_wheel_steering" />
@@ -182,5 +182,5 @@
         </inertial>
     </link>
-    <joint name="front_right_wheel_joint" type="continuous">
+    <joint name="front_right_wheel_joint" type="fixed">
         <origin xyz="0 0 0" rpy="0 0 0" />
         <parent link="right_wheel_steering" />

Commit message: changes to fix broken logic for joint states

File: isaac_ros-dev/src/agv_car_description/description/agv_car.xacro (robot description, xacro)
@@ -250,4 +250,10 @@
             </material>
         </visual>
+        <inertial>
+        <mass value="0.1"/>
+        <origin xyz="0 0 0" rpy="0 0 0"/>
+        <inertia ixx="1e-5" iyy="1e-5" izz="1e-5"
+                ixy="0.0" ixz="0.0" iyz="0.0"/>
+        </inertial>
     </link>
     <joint name="lidar_joint" type="fixed">
