Commit message: Test

File: isaac_ros-dev/src/agv_car_description/description/agv_car2.xacro (robot description, xacro)
@@ -1,55 +1,54 @@
 <?xml version="1.0"?>
 <robot name="ackermann_drive" xmlns:xacro="http://ros.org/wiki/xacro">
-        <!-- Define robot constants -->
-    <xacro:property name="base_width" value="0.92"/>
-    <xacro:property name="base_length" value="1.65"/>
-    <xacro:property name="base_height" value="1.13"/>
-    <xacro:property name="wheel_radius" value="0.2"/>
-    <xacro:property name="front_wheel_width" value="0.15"/>
+    <xacro:property name="base_width" value="1.041"/>
+    <xacro:property name="base_length" value="1.892"/>
+    <xacro:property name="base_height" value="0.626"/>
+    <xacro:property name="front_wheel_radius" value="0.2"/>
+    <xacro:property name="front_wheel_width" value="0.13"/>
+    <xacro:property name="rear_wheel_radius" value="0.2"/>
     <xacro:property name="rear_wheel_width" value="0.17"/>
-    <xacro:property name="front_wheel_ygap" value="0.12"/>
-    <xacro:property name="rear_wheel_ygap" value="0.15"/>
-    <xacro:property name="wheel_zoff" value="0.123"/>
-    <xacro:property name="front_wheel_xoff" value="0.6"/>
-    <xacro:property name="rear_wheel_xoff" value="0.45"/>
+    <xacro:include filename="inertia_macros2.xacro"/>
+    <!-- Colors -->
+    <material name="White">
+        <color rgba="1.0 1.0 1.0 1.0"/>
+    </material>
+    <material name="Blue">
+        <color rgba="0.0 0.0 1.0 1.0"/>
+    </material>
+    <material name="Gray">
+        <color rgba="0.5 0.5 0.5 1.0"/>
+    </material>
     <material name="Black">
-    <color rgba="0 0 0 1" />
-    </material>
-    <material name="Grey">
-        <color rgba="0.8 0.8 0.8 1" />
-    </material>
-    <material name="Orange">
-        <color rgba="1 0.6 0 1" />
-    </material>
-    <material name="White">
-        <color rgba="1 1 1 1" />
-    </material>
-    <link name="base_link" />
+        <color rgba="0.1 0.1 0.1 1"/>
+    </material>
+    <material name="Cyan">
+        <color rgba="0 1.0 1.0 1.0"/>
+    </material>
+    <material name="Red">
+        <color rgba="1 0 0 1.0"/>
+    </material>
+    <link name="base_link"/>
     <!-- Chassis -->
     <link name="chassis">
         <visual>
-        <origin xyz="0 0 0" rpy="0 0 ${pi}" />
-         <geometry>
-                <mesh filename="package://agv_car_description/meshes/new_car_chassis.stl"/>
-            </geometry>
-            <material name="Cyan">
-                <color rgba="0 1.0 1.0 1.0"/>
-            </material>
-        </visual>
-        <collision>
-            <origin xyz=".946 .512 -.313" rpy="0 0 ${pi}" />
+        <origin xyz="0 -0.01 0" rpy="0 0 0" />
+            <geometry>
+                <mesh filename="package://agv_car_description/meshes/new_car_chassis.stl" scale="0.58 0.5 0.58"/>
+            </geometry>
+            <material name="Blue"/>
+        </visual>
+        <collision>
+            <!-- <origin xyz="0 -0.01 0" rpy="0 0 0" />
                 <geometry>
-                    <mesh filename="package://agv_car_description/meshes/agv_chassis.stl"/>
-                </geometry>
-        </collision>
-        <!-- <xacro:box_inertia m="15" w="${base_width}" d="${base_length}" h="${base_height}"/> -->
-        <inertial>
-        <origin xyz="0 0 0" rpy="0 0 0" />
-        <mass value="100" />
-        <inertia ixx="10.4" ixy="0.0" ixz="0.0" iyy="35.4" iyz="0.0" izz="41.66" />
-        </inertial>
+                    <mesh filename="package://robot_description/description/meshes/new_car_chassis.stl" scale="0.58 0.58 0.58"/>
+                </geometry> -->
+        </collision>
+        <!-- make box slightly smaller than actual to prevent accidental self collision y=0.92-->
+        <xacro:inertia_box mass="150" x="1.65" y="0.92" z="1.13">
+            <origin rpy="0 -0.01 0" xyz="0 0 0"/>
+        </xacro:inertia_box>
     </link>
     <joint name="chassis_joint" type="fixed">
-        <origin xyz="0 0 .313" rpy="0 0 0" />
+        <origin xyz="0 0 0.2" rpy="0 0 0" />
         <parent link="base_link" />
         <child link="chassis" />
@@ -58,26 +57,25 @@
     <link name="rear_left_wheel">
         <visual>
-            <geometry>
-                <cylinder radius="${wheel_radius}" length="${rear_wheel_width}"/>
-            </geometry>
-            <material name="Gray">
-                <color rgba="0.5 0.5 0.5 1.0"/>
-            </material>
-        </visual>
-            <collision>
-                <geometry>
-                    <cylinder radius="${wheel_radius}" length="${rear_wheel_width}"/>
-                </geometry>
-            </collision>
-        <inertial>
-        <mass value="11.3" />
-        <inertia ixx="0.26" ixy="0.0" ixz="0.0" iyy="0.26" iyz="0.0" izz="0.51" />
-        </inertial>
+            <origin rpy="1.57 0 0"/>
+            <geometry>
+                <cylinder radius="${rear_wheel_radius}" length="${rear_wheel_width}"/>
+            </geometry>
+            <material name="Black"/>
+        </visual>
+        <collision>
+            <origin rpy="1.57 0 0"/>
+            <geometry>
+                <cylinder radius="${rear_wheel_radius}" length="${rear_wheel_width}"/>
+            </geometry>
+        </collision>
+        <xacro:inertia_cylinder mass="6.8" length="0.17" radius="0.2">
+            <origin xyz="-0.6 0.42 0" rpy="-1.57 0 0"/>
+        </xacro:inertia_cylinder>
     </link>
     <joint name="rear_left_wheel_joint" type="fixed">
-        <origin xyz="-0.9 0.5 -0.2" rpy="-1.57 0 0" />
+        <origin xyz="-0.6 0.42 0" rpy="0 0 0"/>
         <parent link="chassis" />
         <child link="rear_left_wheel" />
-        <axis xyz="0 0 1" />
+        <axis xyz="0 1 0" />
         <dynamics damping="0.2" />
     </joint>
@@ -85,26 +83,25 @@
     <link name="rear_right_wheel">
         <visual>
-            <geometry>
-                <cylinder radius="${wheel_radius}" length="${rear_wheel_width}"/>
-            </geometry>
-            <material name="Gray">
-                <color rgba="0.5 0.5 0.5 1.0"/>
-            </material>
-        </visual>
-            <collision>
-                <geometry>
-                    <cylinder radius="${wheel_radius}" length="${rear_wheel_width}"/>
-                </geometry>
-            </collision>
-        <inertial>
-        <mass value="11.3" />
-        <inertia ixx="0.26" ixy="0.0" ixz="0.0" iyy="0.26" iyz="0.0" izz="0.51" />
-        </inertial>
+            <origin rpy="1.57 0 0"/>
+            <geometry>
+                <cylinder radius="${rear_wheel_radius}" length="${rear_wheel_width}"/>
+            </geometry>
+            <material name="Black"/>
+        </visual>
+        <collision>
+            <origin rpy="1.57 0 0"/>
+            <geometry>
+                <cylinder radius="${rear_wheel_radius}" length="${rear_wheel_width}"/>
+            </geometry>
+        </collision>
+        <xacro:inertia_cylinder mass="6.8" length="0.17" radius="0.2">
+            <origin xyz="-0.6 -0.42 0" rpy="-1.57 0 0" />
+        </xacro:inertia_cylinder>
     </link>
     <joint name="rear_right_wheel_joint" type="fixed">
-        <origin xyz="-0.9 -0.5 -0.2" rpy="-1.57 0 0" />
+        <origin xyz="-0.6 -0.42 0" rpy="0 0 0" />
         <parent link="chassis" />
         <child link="rear_right_wheel" />
-        <axis xyz="0 0 1" />
+        <axis xyz="0 1 0" />
         <dynamics damping="0.2" />
     </joint>
@@ -112,50 +109,51 @@
     <link name="left_wheel_steering">
         <inertial>
-        <mass value="0.1"/>
-        <inertia ixx="0" ixy="0.0" ixz="0.0" iyy="0.0" iyz="0.0" izz="0.0" />
+            <mass value="0.1"/>
+            <inertia ixx="0" ixy="0.0" ixz="0.0" iyy="0.0" iyz="0.0" izz="0.0" />
         </inertial>
     </link>
     <joint name="left_wheel_steering_joint" type="fixed">
-        <origin xyz="0.9 0.5 -0.2" rpy="1.57 0 0" />
-        <parent link="chassis" />
-        <child link="left_wheel_steering" />
-        <axis xyz="0 1 0" />
-        <dynamics damping="0.2" />
-        <limit effort="1000.0" lower="-1.57" upper="1.57" velocity="30"/>
+        <origin xyz="0.6 0.45 0" rpy="0 0 0"/>
+        <parent link="chassis"/>
+        <child link="left_wheel_steering"/>
+        <axis xyz="0 0 1"/>
+        <dynamics damping="0.2"/>
+        <!-- effort = torque (N/m) Lower/upper = steering angle rad-->
+        <limit effort="100.0" lower="-0.785" upper="0.785" velocity="30"/>
     </joint>
     <!-- right steer Link -->
     <link name="right_wheel_steering">
         <inertial>
-        <mass value="0.1"/>
-        <inertia ixx="0" ixy="0.0" ixz="0.0" iyy="0.0" iyz="0.0" izz="0.0" />
+            <mass value="0.1"/>
+            <inertia ixx="0" ixy="0.0" ixz="0.0" iyy="0.0" iyz="0.0" izz="0.0" />
         </inertial>
     </link>
     <joint name="right_wheel_steering_joint" type="fixed">
-        <origin xyz="0.9 -0.5 -0.2" rpy="1.57 0 0" />
-        <parent link="chassis" />
-        <child link="right_wheel_steering" />
-        <axis xyz="0 1 0" />
-        <dynamics damping="0.2" />
-        <limit effort="1000.0" lower="-1.57" upper="1.57" velocity="30"/>
+        <origin xyz="0.6 -0.45 0" rpy="0 0 0"/>
+        <parent link="chassis"/>
+        <child link="right_wheel_steering"/>
+        <axis xyz="0 0 1"/>
+        <dynamics damping="0.2"/>
+        <!-- effort = torque (N/m) Lower/upper = steering angle rad-->
+        <limit effort="100.0" lower="-0.785" upper="0.785" velocity="30"/>
     </joint>
     <!-- front left wheel Link -->
     <link name="front_left_wheel">
          <visual>
-            <geometry>
-                <cylinder radius="${wheel_radius}" length="${front_wheel_width}"/>
-            </geometry>
-            <material name="Gray">
-                <color rgba="0.5 0.5 0.5 1.0"/>
-            </material>
-        </visual>
-            <collision>
-                <geometry>
-                    <cylinder radius="${wheel_radius}" length="${front_wheel_width}"/>
-                </geometry>
-            </collision>
-        <inertial>
-        <mass value="11.3" />
-        <inertia ixx="0.26" ixy="0.0" ixz="0.0" iyy="0.26" iyz="0.0" izz="0.51" />
-        </inertial>
+            <origin rpy="1.57 0 0"/>
+            <geometry>
+                <cylinder radius="${front_wheel_radius}" length="${front_wheel_width}"/>
+            </geometry>
+            <material name="Black"/>
+        </visual>
+        <collision>
+            <origin rpy="1.57 0 0"/>
+            <geometry>
+                <cylinder radius="${front_wheel_radius}" length="${front_wheel_width}"/>
+            </geometry>
+        </collision>
+        <xacro:inertia_cylinder mass="4.5" length="0.13" radius="0.2">
+            <origin xyz="0.6 0.45 0" rpy="1.57 0 0"/>
+        </xacro:inertia_cylinder>
     </link>
     <joint name="front_left_wheel_joint" type="fixed">
@@ -163,5 +161,5 @@
         <parent link="left_wheel_steering" />
         <child link="front_left_wheel" />
-        <axis xyz="0 0 1" />
+        <axis xyz="0 1 0" />
         <dynamics damping="0.2" />
     </joint>
@@ -169,20 +167,19 @@
     <link name="front_right_wheel">
         <visual>
-            <geometry>
-                <cylinder radius="${wheel_radius}" length="${front_wheel_width}"/>
-            </geometry>
-            <material name="Gray">
-                <color rgba="0.5 0.5 0.5 1.0"/>
-            </material>
-        </visual>
-            <collision>
-                <geometry>
-                    <cylinder radius="${wheel_radius}" length="${front_wheel_width}"/>
-                </geometry>
-            </collision>
-        <inertial>
-        <mass value="11.3" />
-        <inertia ixx="0.26" ixy="0.0" ixz="0.0" iyy="0.26" iyz="0.0" izz="0.51" />
-        </inertial>
+            <origin rpy="1.57 0 0"/>
+            <geometry>
+                <cylinder radius="${front_wheel_radius}" length="${front_wheel_width}"/>
+            </geometry>
+            <material name="Black"/>
+        </visual>
+        <collision>
+            <origin rpy="1.57 0 0"/>
+            <geometry>
+                <cylinder radius="${front_wheel_radius}" length="${front_wheel_width}"/>
+            </geometry>
+        </collision>
+        <xacro:inertia_cylinder mass="4.5" length="0.13" radius="0.2">
+            <origin xyz="0.6 -0.45 0" rpy="1.57 0 0"/>
+        </xacro:inertia_cylinder>
     </link>
     <joint name="front_right_wheel_joint" type="fixed">
@@ -190,47 +187,21 @@
         <parent link="right_wheel_steering" />
         <child link="front_right_wheel" />
-        <axis xyz="0 0 1" />
-        <dynamics damping="0.2" />
-    </joint>
-     <!-- <link name="virtual_front_wheel">
-    <visual>
-        <origin xyz="0 0 0" rpy="0 0 0"/>
-        <geometry>
-        <cylinder length="0.01" radius="${wheel_radius}"/>
-        </geometry>
-    </visual>
-    </link>
-    <joint name="virtual_front_wheel_joint" type="revolute">
-    <parent link="chassis"/>
-    <child link="virtual_front_wheel"/>
-    <origin xyz="0.9 0 -0.2" rpy="1.57 0 0"/>
-    <axis xyz="0 1 0"/>
-    <limit lower="-0.7853" upper="0.7853" effort="100.0" velocity="100.0"/>
-    <dynamics damping="0.2"/>
-    </joint> -->
-    <!-- virtual rear wheel -->
-    <!-- <link name="virtual_rear_wheel">
-    <visual>
-        <origin xyz="0 0 0" rpy="0 0 0"/>
-        <geometry>
-        <cylinder length="0.01" radius="${wheel_radius}"/>
-        </geometry>
-    </visual>
-    </link> -->
-    <!-- <joint name="virtual_rear_wheel_joint" type="continuous">
-    <parent link="chassis"/>
-    <child link="virtual_rear_wheel"/>
-    <origin xyz="-0.9 0 -0.2" rpy="-1.57 0 0"/>
-    <axis xyz="0 0 1"/>
-    <limit effort="100.0" velocity="100.0"/>
-    <dynamics damping="0.2"/>
-    </joint> -->
-        <!-- IMU and GPS combined sensor -->
-    <link name="imu_link"/>
-    <joint name="imu_joint" type="fixed">
-    <parent link="chassis"/>
-    <child link="imu_link"/>
-    <!-- Adjust this to the actual mounting point on your robot -->
-    <origin xyz="0 0 1.2" rpy="0 0 0"/>
+        <axis xyz="0 1 0" />
+        <dynamics damping="0.2" />
+    </joint>
+    <!-- IMU -->
+    <link name="imu_link">
+        <pose>0 0 0 0 0 0</pose>  <!-- Adjust height based on your vehicle -->
+        <visual>
+            <geometry>
+                <box size ="0.05 0.05 0.01"/>
+            </geometry>
+            <material name ="White"/>
+        </visual>
+    </link>
+     <joint name="imu_joint" type="fixed">
+        <origin xyz="0 0 1" rpy="0 0 0" />
+        <parent link="chassis" />
+        <child link="imu_link" />
     </joint>
     <link name="gps_link"/>
@@ -239,8 +210,7 @@
     <child link="gps_link"/>
     <!-- Same origin as imu_link -->
-    <origin xyz="0 0 1.2" rpy="0 0 0"/>
-    </joint>
-        <!-- Lidar -->
-    <link name="lidar">
+    <origin xyz="0 0 1" rpy="0 0 0"/>
+    </joint>
+     <link name="lidar">
         <visual>
             <origin xyz="0 0 0" rpy="0 0 0"/>
